File: esp32-pcie-card-hw/pci-e_connector.sch (KiCad schematic (older format))
At the start: 1 part

Commit message: WIP
Parts:
- J2: renamed from J?; footprint (none) -> mpcie:mini-PCIe_F1_Full
Changed lines of the file:
@@
 $EndDescr
 $Comp
-L mpcie:miniPCIe J?
+L mpcie:miniPCIe J2
 U 1 1 60C40758
 P 5850 3750
-F 0 "J?" H 5850 5287 60  0000 C CNN
+F 0 "J2" H 5850 5287 60  0000 C CNN
 F 1 "miniPCIe" H 5850 5181 60  0000 C CNN
-F 2 "" H 6950 1650 60  0001 C CNN
+F 2 "mpcie:mini-PCIe_F1_Full" H 6950 1650 60  0001 C CNN
 F 3 "https://pcisig.com/specifications/pciexpress/base" H 6950 1650 60  0001 C CNN
 	1    5850 3750
