File: esp32-pcie-card-hw/usb-serial.sch (KiCad schematic (older format))
At the start: 14 parts, among them Q1 MBT2222ADW1T1

Commit message: WIP on schematics
Changed lines of the file:
@@
 encoding utf-8
 Sheet 4 4
-Title ""
-Date ""
+Title "USB to Serial Converter"
+Date "2021-02-28"
 Rev ""
-Comp ""
+Comp "Pedro Minatel"
 Comment1 ""
 Comment2 ""
@@
 Wire Wire Line
 	7550 3500 7650 3500
-Text Notes 3400 1450 0    79   Italic 0
+Text Notes 500  650  0    79   Italic 0
 USB to Serial Interface and USB Type C Connector
 $Comp

Commit message: WIP
Parts:
- gave numbers to parts that had none: 1
Changed lines of the file:
@@
 $EndComp
 $Comp
-L Interface_USB:CP2102N-Axx-xQFN28 U?
+L Interface_USB:CP2102N-Axx-xQFN28 U1
 U 1 1 60BDDEFC
 P 5800 4900
-F 0 "U?" H 6250 6200 50  0000 C CNN
+F 0 "U1" H 6250 6200 50  0000 C CNN
 F 1 "CP2102N-Axx-xQFN28" H 6300 3600 50  0000 C CNN
 F 2 "Package_DFN_QFN:QFN-28-1EP_5x5mm_P0.5mm_EP3.35x3.35mm" H 7100 3650 50  0001 C CNN
@@
 	3900 4300 5300 4300
 $Comp
-L power:+3V3 #PWR?
+L power:+3V3 #PWR0109
 U 1 1 60C6B856
 P 3900 3850
-F 0 "#PWR?" H 3900 3700 50  0001 C CNN
+F 0 "#PWR0109" H 3900 3700 50  0001 C CNN
 F 1 "+3V3" H 3915 4023 50  0000 C CNN
 F 2 "" H 3900 3850 50  0001 C CNN
